File: src/babelbabel.brd (EAGLE design)
At the start: 41 x 75.5 mm, 144 parts, among them CON1 CON-4P-TABS-JST_GH-RA, CON10 CON-6P-SM06B, CON101 PINHEAD_1X04-2.54, CON102 PINHEAD_1X03-2.54, CON11 PINHEAD_1X04-2.54, CON12 PINHEAD_1X06-2.54, CON15 PINHEAD_1X04-2.54, CON16 CON-4P-TABS-JST_GH-RA, CON2 PINHEAD_1X04-2.54, CON201 PINHEAD_1X04-2.54, CON202 PINHEAD_1X03-2.54, CON3 PINHEAD_1X04-2.54, CON4 USB-AA-PTH, CON5 CON-4P-TABS-JST_GH-RA, CON6 CON-4P-TABS-JST_GH-RA, CON7 USB-1, IC101 STM32F373CBT6-LQFP48, IC102 STM32F373RCT6, IC103 AP2127-3.3, IC105 TJA1051-SO8, IC108 TPD3S014DBVR-SOT23-6, IC13 STM32F103CBT7, IC14 74LVC2T45, IC15 74LVC2T45, IC16 74LVC2T45, IC17 74LVC2T45, IC201 STM32F373CBT6-LQFP48, IC202 STM32F373RCT6, IC203 AP2127-3.3, IC205 TJA1051-SO8, IC208 TPD3S014DBVR-SOT23-6, IC3 AP2127-3.3, IC9 FE1.1S, J1 CONNECTION-SMD, J2 CONNECTION-SMD, Q101 16MHz, Q102 2N7002, Q201 16MHz, Q202 2N7002, Q7 8MHz, Q8 12MHz, Q9 NTZD3152PT1G

Commit message: Minor tweaks
Connections:
- net N$6 renamed CANH2
Routing:
- net GND: vias 117 -> 115
Changed lines of the file:
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@@
 <grid distance="0.05" unitdist="mm" unit="mm" style="lines" multiple="1" display="yes" altdistance="5" altunitdist="mil" altunit="mil"/>
 <layers>
-<layer number="1" name="Top" color="4" fill="1" visible="no" active="yes"/>
+<layer number="1" name="Top" color="4" fill="1" visible="yes" active="yes"/>
 <layer number="2" name="Route2" color="16" fill="1" visible="no" active="yes"/>
 <layer number="3" name="Route3" color="17" fill="1" visible="no" active="no"/>
@@
 <layer number="14" name="Route14" color="22" fill="1" visible="no" active="no"/>
 <layer number="15" name="Route15" color="23" fill="1" visible="no" active="yes"/>
-<layer number="16" name="Bottom" color="1" fill="1" visible="yes" active="yes"/>
+<layer number="16" name="Bottom" color="1" fill="1" visible="no" active="yes"/>
 <layer number="17" name="Pads" color="2" fill="1" visible="yes" active="yes"/>
 <layer number="18" name="Vias" color="2" fill="1" visible="yes" active="yes"/>
 <layer number="19" name="Unrouted" color="6" fill="1" visible="yes" active="yes"/>
 <layer number="20" name="Dimension" color="24" fill="1" visible="yes" active="yes"/>
-<layer number="21" name="tPlace" color="7" fill="1" visible="no" active="yes"/>
-<layer number="22" name="bPlace" color="7" fill="1" visible="yes" active="yes"/>
-<layer number="23" name="tOrigins" color="15" fill="1" visible="no" active="yes"/>
-<layer number="24" name="bOrigins" color="15" fill="1" visible="yes" active="yes"/>
-<layer number="25" name="tNames" color="7" fill="1" visible="no" active="yes"/>
-<layer number="26" name="bNames" color="7" fill="1" visible="yes" active="yes"/>
+<layer number="21" name="tPlace" color="7" fill="1" visible="yes" active="yes"/>
+<layer number="22" name="bPlace" color="7" fill="1" visible="no" active="yes"/>
+<layer number="23" name="tOrigins" color="15" fill="1" visible="yes" active="yes"/>
+<layer number="24" name="bOrigins" color="15" fill="1" visible="no" active="yes"/>
+<layer number="25" name="tNames" color="7" fill="1" visible="yes" active="yes"/>
+<layer number="26" name="bNames" color="7" fill="1" visible="no" active="yes"/>
 <layer number="27" name="tValues" color="7" fill="1" visible="no" active="yes"/>
 <layer number="28" name="bValues" color="7" fill="1" visible="no" active="yes"/>
@@
 <layer number="49" name="Reference" color="7" fill="1" visible="yes" active="yes"/>
 <layer number="50" name="dxf" color="7" fill="1" visible="no" active="no"/>
-<layer number="51" name="tDocu" color="7" fill="1" visible="no" active="yes"/>
-<layer number="52" name="bDocu" color="7" fill="1" visible="yes" active="yes"/>
+<layer number="51" name="tDocu" color="7" fill="1" visible="yes" active="yes"/>
+<layer number="52" name="bDocu" color="7" fill="1" visible="no" active="yes"/>
 <layer number="53" name="tGND_GNDA" color="7" fill="9" visible="no" active="no"/>
 <layer number="54" name="bGND_GNDA" color="1" fill="9" visible="no" active="no"/>
@@
 </layers>
 <board>
-<fusionsync huburn="a.cGVyc29uYWw6dWUyYWE4ZDY4" projecturn="a.cGVyc29uYWw6dWUyYWE4ZDY4IzIwMTgxMTAxMTU3ODkyNjgx" f3durn="urn:adsk.wipprod:dm.lineage:kGuPgqnzRmWLHCf0r-cvPw" pcbguid="" lastpulledtime="" lastsyncedchangeguid="" latestrevisionid="c319dde0-590c-43ad-b738-9d1c039037c4" lastsyncedrevisionid="c319dde0-590c-43ad-b738-9d1c039037c4" lastboardhashguid="029d2627-3a96-b5a4-349e-fa68dd392475" lastpushedtime="2020-12-25T18:48:24Z" linktopcb3d="true"/>
+<fusionsync huburn="a.cGVyc29uYWw6dWUyYWE4ZDY4" projecturn="a.cGVyc29uYWw6dWUyYWE4ZDY4IzIwMTgxMTAxMTU3ODkyNjgx" f3durn="urn:adsk.wipprod:dm.lineage:kGuPgqnzRmWLHCf0r-cvPw" pcbguid="" lastpulledtime="" lastsyncedchangeguid="" latestrevisionid="41216dde-41be-4269-847a-d92c805843a9" lastsyncedrevisionid="41216dde-41be-4269-847a-d92c805843a9" lastboardhashguid="f66e5044-090c-3d7d-41af-6c733bc627cd" lastpushedtime="2020-12-28T11:51:55Z" linktopcb3d="true"/>
 <plain>
 <wire x1="41" y1="33.75" x2="41" y2="32.35" width="0.01" layer="49"/>
@@
 <attribute name="MANF" value="" x="-34.1" y="3.15" size="1.778" layer="27" rot="R270" display="off"/>
 <attribute name="MANF#" value="" x="-34.1" y="3.15" size="1.778" layer="27" rot="R270" display="off"/>
-<attribute name="NAME" x="23.05" y="-26.85" size="0.5" layer="25" font="vector" ratio="15" rot="R270" align="center"/>
+<attribute name="NAME" x="20.9" y="-26.85" size="0.508" layer="25" font="vector" ratio="15" rot="R270" align="center"/>
 </element>
 <element name="C117" library="rc" library_urn="urn:adsk.eagle:library:2539423" package="C0402" package3d_urn="urn:adsk.eagle:package:2539461/2" value="20pF" x="21.1" y="-29.65" smashed="yes">
@@
 <attribute name="MANF" value="" x="18.4" y="7" size="1.778" layer="27" rot="R90" display="off"/>
 <attribute name="MANF#" value="" x="18.4" y="7" size="1.778" layer="27" rot="R90" display="off"/>
-<attribute name="NAME" x="18.4" y="7" size="1" layer="25" font="vector" ratio="15" rot="R90" align="center"/>
+<attribute name="NAME" x="18.4" y="7" size="0.508" layer="25" font="vector" ratio="15" rot="R90" align="center"/>
 </element>
 <element name="C38" library="rc" library_urn="urn:adsk.eagle:library:2539423" package="C0402" package3d_urn="urn:adsk.eagle:package:2539461/2" value="10pF" x="18.8" y="4.2" smashed="yes" rot="R180">
@@
 <attribute name="MANF" value="" x="-34.1" y="21.15" size="1.778" layer="27" rot="R270" display="off"/>
 <attribute name="MANF#" value="" x="-34.1" y="21.15" size="1.778" layer="27" rot="R270" display="off"/>
-<attribute name="NAME" x="23.05" y="-8.85" size="0.5" layer="25" font="vector" ratio="15" rot="R270" align="center"/>
+<attribute name="NAME" x="20.9" y="-8.85" size="0.508" layer="25" font="vector" ratio="15" rot="R270" align="center"/>
 </element>
 <element name="C217" library="rc" library_urn="urn:adsk.eagle:library:2539423" package="C0402" package3d_urn="urn:adsk.eagle:package:2539461/2" value="20pF" x="21.1" y="-11.65" smashed="yes">
@@
 <contactref element="IC102" pad="31"/>
 <contactref element="CON101" pad="1"/>
-<via x="14.65" y="-24.6" extent="1-16" drill="0.3" diameter="0.6"/>
 <via x="14.25" y="-28.4" extent="1-16" drill="0.3" diameter="0.6"/>
 <via x="9.45" y="-22.5" extent="1-16" drill="0.3" diameter="0.6"/>
@@
 <contactref element="IC202" pad="31"/>
 <contactref element="CON201" pad="1"/>
-<via x="14.65" y="-6.6" extent="1-16" drill="0.3" diameter="0.6"/>
 <via x="14.25" y="-10.4" extent="1-16" drill="0.3" diameter="0.6"/>
 <via x="9.45" y="-4.5" extent="1-16" drill="0.3" diameter="0.6"/>
@@
 </polygon>
 <polygon width="0.2" layer="15" thermals="no">
-<vertex x="15.4" y="-28.95"/>
-<vertex x="15.4" y="-29.45"/>
-<vertex x="16.3" y="-29.45"/>
-<vertex x="16.3" y="-28.95"/>
+<vertex x="15.35" y="-28.95"/>
+<vertex x="15.35" y="-29.45"/>
+<vertex x="16.35" y="-29.45"/>
+<vertex x="16.35" y="-28.95"/>
 </polygon>
-<wire x1="14.65" y1="-23.8" x2="15.16924375" y2="-23.8" width="0.5" layer="15"/>
-<wire x1="15.16924375" y1="-23.8" x2="16.15" y2="-24.78075625" width="0.5" layer="15"/>
-<wire x1="16.15" y1="-24.78075625" x2="16.15" y2="-29.2" width="0.5" layer="15"/>
+<wire x1="14.65" y1="-23.8" x2="15.5" y2="-24.65" width="0.5" layer="15"/>
+<wire x1="16.15" y1="-29.2" x2="15.5" y2="-29.2" width="0.5" layer="15"/>
+<wire x1="15.5" y1="-24.65" x2="15.5" y2="-29.2" width="0.5" layer="15"/>
 <wire x1="2" y1="-20.94" x2="2.76" y2="-21.7" width="0.3" layer="1"/>
 <wire x1="2.76" y1="-21.7" x2="6" y2="-21.7" width="0.3" layer="1"/>
@@
 <wire x1="16.1" y1="-7.2" x2="14.1" y2="-7.2" width="0.2" layer="2"/>
 </signal>
-<signal name="N$6">
+<signal name="CANH2">
 <contactref element="S3" pad="1"/>
 <contactref element="CON2" pad="2"/>
@@
 </polygon>
 <polygon width="0.2" layer="15" thermals="no">
-<vertex x="15.4" y="-10.95"/>
-<vertex x="15.4" y="-11.45"/>
-<vertex x="16.3" y="-11.45"/>
-<vertex x="16.3" y="-10.95"/>
+<vertex x="15.35" y="-10.95"/>
+<vertex x="15.35" y="-11.45"/>
+<vertex x="16.35" y="-11.45"/>
+<vertex x="16.35" y="-10.95"/>
 </polygon>
-<wire x1="14.65" y1="-5.8" x2="15.16924375" y2="-5.8" width="0.5" layer="15"/>
-<wire x1="15.16924375" y1="-5.8" x2="16.15" y2="-6.78075625" width="0.5" layer="15"/>
-<wire x1="16.15" y1="-6.78075625" x2="16.15" y2="-11.2" width="0.5" layer="15"/>
+<wire x1="14.65" y1="-5.8" x2="15.5" y2="-6.65" width="0.5" layer="15"/>
+<wire x1="15.5" y1="-6.65" x2="15.5" y2="-11.2" width="0.5" layer="15"/>
+<wire x1="15.5" y1="-11.2" x2="16.15" y2="-11.2" width="0.5" layer="15"/>
 <wire x1="6" y1="-3.7" x2="2.885" y2="-3.7" width="0.3" layer="1"/>
 <wire x1="2.885" y1="-3.7" x2="2.125" y2="-2.94" width="0.3" layer="1"/>
