File: src/part B1.brd (EAGLE design)
At the start: 41 x 75.5 mm, 0 parts

Commit message: ready for review
Other:
- outline, holes or cut-outs redrawn
Changed lines of the file:
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@@
 <text x="1" y="11" size="2.5" layer="21" font="vector" ratio="15" rot="R90" align="top-center">BABEL 1</text>
 <text x="1" y="29" size="2.5" layer="21" font="vector" ratio="15" rot="R90" align="top-center">BABEL 2</text>
-<text x="1" y="47" size="2.5" layer="21" font="vector" ratio="15" rot="R90" align="top-center">Dronecode
-probe</text>
+<text x="1" y="53" size="2.5" layer="21" font="vector" ratio="15" rot="R90" align="top-center">Dronecode probe</text>
 <wire x1="-2" y1="38" x2="33" y2="38" width="0.3" layer="21"/>
 <wire x1="-2" y1="20" x2="33" y2="20" width="0.3" layer="21"/>
@@
 <wire x1="31.3" y1="38.7" x2="21.4" y2="38.7" width="0.2" layer="21"/>
 <text x="8.7" y="70.1" size="2.5" layer="21" font="vector" ratio="15" align="center">To PC</text>
-<text x="23" y="61" size="2.5" layer="21" font="vector" ratio="15" rot="R90" align="center">To device</text>
+<text x="23.2" y="65.2" size="2.5" layer="21" font="vector" ratio="15" rot="R270" align="center">To device</text>
 <text x="26.4" y="14.5" size="1.5" layer="21" font="vector" ratio="15" align="center-left">GND
 CAN L
@@
 <vertex x="30.2" y="6.4"/>
 </polygon>
-<wire x1="7" y1="53.2" x2="11" y2="53.2" width="0.1016" layer="21"/>
-<wire x1="11" y1="53.2" x2="11" y2="52.2" width="0.1016" layer="21"/>
-<wire x1="11" y1="52.2" x2="7" y2="52.2" width="0.1016" layer="21"/>
+<wire x1="7" y1="53.2" x2="10.1" y2="53.2" width="0.1016" layer="21"/>
+<wire x1="10.1" y1="53.2" x2="10.1" y2="52.2" width="0.1016" layer="21"/>
+<wire x1="10.1" y1="52.2" x2="7" y2="52.2" width="0.1016" layer="21"/>
 <wire x1="7" y1="52.2" x2="7" y2="53.2" width="0.1016" layer="21"/>
-<text x="12.5" y="54.4" size="1.5" layer="21" font="vector" ratio="15" align="center-right">status</text>
+<text x="11.2" y="51.1" size="1.5" layer="21" font="vector" ratio="15" align="center-right">status</text>
 <polygon width="0.1" layer="30">
 <vertex x="7" y="53.2"/>
-<vertex x="11" y="53.2"/>
-<vertex x="11" y="52.2"/>
+<vertex x="10.1" y="53.2"/>
+<vertex x="10.1" y="52.2"/>
 <vertex x="7" y="52.2"/>
 </polygon>
 <polygon width="0.1" layer="29">
 <vertex x="7" y="53.2"/>
-<vertex x="11" y="53.2"/>
-<vertex x="11" y="52.2"/>
+<vertex x="10.1" y="53.2"/>
+<vertex x="10.1" y="52.2"/>
 <vertex x="7" y="52.2"/>
 </polygon>
@@
 <text x="14.7" y="32.5" size="1.5" layer="21" font="vector" ratio="15" align="center">OFF</text>
 <text x="14.6" y="14.3" size="1.5" layer="21" font="vector" ratio="15" align="center">OFF</text>
+<wire x1="21.7" y1="52.4" x2="21.7" y2="55.5" width="0.01" layer="20"/>
+<wire x1="21.7" y1="55.5" x2="21.1" y2="56.2" width="0.01" layer="20" curve="90"/>
+<wire x1="21.1" y1="56.2" x2="11.3" y2="56.2" width="0.01" layer="20"/>
+<wire x1="11.3" y1="56.2" x2="10.6" y2="55.7" width="0.01" layer="20" curve="90"/>
+<wire x1="10.6" y1="55.7" x2="10.6" y2="52.6" width="0.01" layer="20"/>
+<wire x1="10.6" y1="52.6" x2="11.2" y2="51.95" width="0.01" layer="20" curve="90"/>
+<wire x1="11.2" y1="51.95" x2="21" y2="51.95" width="0.01" layer="20"/>
+<wire x1="21" y1="51.95" x2="21.7" y2="52.4" width="0.01" layer="20" curve="90"/>
+<text x="20.3" y="57.1" size="1.5" layer="21" font="vector" ratio="15" align="center">ON</text>
+<text x="12.1" y="57.1" size="1.5" layer="21" font="vector" ratio="15" align="center">OFF</text>
 </plain>
 <attributes>
@@
 <polygon width="0.1" layer="1" pour="cutout">
 <vertex x="7" y="53.2"/>
-<vertex x="11" y="53.2"/>
-<vertex x="11" y="52.2"/>
+<vertex x="10.1" y="53.2"/>
+<vertex x="10.1" y="52.2"/>
 <vertex x="7" y="52.2"/>
 </polygon>
